Commit message: Added turtlebot meshes and showing it in RVIZ

File: nuturtle_description/urdf/turtlebot3_burger.urdf.xacro (robot description, xacro)
@@ -2,5 +2,5 @@
 <!-- This code was modified from the ROBOTIS-GIT turtlebot3 Package
 01/07/2023
-https://github.com/ROBOTIS-GIT/turtlebot3/blob/humble-devel/turtlebot3_description/urdf/turtlebot3_burger.urdf -->
+https://github.com/ROBOTIS-GIT/turtlebot3/blob/humble-devel/nuturtle_description/urdf/turtlebot3_burger.urdf -->
 <robot name="turtlebot3_burger"
   xmlns:xacro="http://ros.org/wiki/xacro">
@@ -46,5 +46,5 @@
       <origin xyz="-0.032 0 0.0" rpy="0 0 0"/>
       <geometry>
-        <mesh filename="package://turtlebot3_description/meshes/bases/burger_base.stl" scale="0.001 0.001 0.001"/>
+        <mesh filename="package://nuturtle_description/meshes/burger_base.stl" scale="0.001 0.001 0.001"/>
       </geometry>
       <material name="light_black"/>
@@ -72,5 +72,5 @@
       <origin xyz="0 0 0" rpy="1.57 0 0"/>
       <geometry>
-        <mesh filename="package://turtlebot3_description/meshes/wheels/left_tire.stl" scale="0.001 0.001 0.001"/>
+        <mesh filename="package://nuturtle_description/meshes/left_tire.stl" scale="0.001 0.001 0.001"/>
       </geometry>
       <material name="dark"/>
@@ -98,5 +98,5 @@
       <origin xyz="0 0 0" rpy="1.57 0 0"/>
       <geometry>
-        <mesh filename="package://turtlebot3_description/meshes/wheels/right_tire.stl" scale="0.001 0.001 0.001"/>
+        <mesh filename="package://nuturtle_description/meshes/right_tire.stl" scale="0.001 0.001 0.001"/>
       </geometry>
       <material name="dark"/>
@@ -147,5 +147,5 @@
       <origin xyz="0 0 0.0" rpy="0 0 0"/>
       <geometry>
-        <mesh filename="package://turtlebot3_description/meshes/sensors/lds.stl" scale="0.001 0.001 0.001"/>
+        <mesh filename="package://nuturtle_description/meshes/lds.stl" scale="0.001 0.001 0.001"/>
       </geometry>
       <material name="dark"/>

Commit message: Added yaml and imported to urdf

File: nuturtle_description/urdf/turtlebot3_burger.urdf.xacro (robot description, xacro)
@@ -5,4 +5,14 @@
 <robot name="turtlebot3_burger"
   xmlns:xacro="http://ros.org/wiki/xacro">
+  <xacro:property name="yaml_file" value="$(find nuturtle_description)/config/diff_params.yaml" />
+  <xacro:property name="props" value="${xacro.load_yaml(yaml_file)}"/>
+  <xacro:property name="star" value="${props['/**']}" />
+  <xacro:property name="ros_parameters" value="${star['ros__parameters']}" />
+  <xacro:property name="wheel_radius" value="${ros_parameters['wheel_radius']}" />
+  <xacro:property name="track_width" value="${ros_parameters['track_width']}" />
+  <xacro:property name="motor_cmd_max" value="${ros_parameters['motor_cmd_max']}" />
+  <xacro:property name="motor_cmd_per_rad_sec" value="${ros_parameters['motor_cmd_per_rad_sec']}" />
+  <xacro:property name="encoder_ticks_per_rad" value="${ros_parameters['encoder_ticks_per_rad']}" />
+  <xacro:property name="collision_radius" value="${ros_parameters['collision_radius']}" />
   <!-- Init colour -->
   <material name="black">
@@ -53,5 +63,10 @@
       <origin xyz="-0.032 0 0.070" rpy="0 0 0"/>
       <geometry>
-        <box size="0.140 0.140 0.143"/>
+        <xacro:if value="${collision_radius &lt; 0}">
+          <box size="0.140 0.140 0.143"/>
+        </xacro:if>
+        <xacro:if value="${collision_radius &gt; 0}">
+          <cylinder length="0.143" radius="${collision_radius}" />
+        </xacro:if>
       </geometry>
     </collision>
@@ -65,5 +80,5 @@
     <parent link="base_link"/>
     <child link="wheel_left_link"/>
-    <origin xyz="0.0 0.08 0.023" rpy="-1.57 0 0"/>
+    <origin xyz="0.0 ${track_width/2} 0.023" rpy="-1.57 0 0"/>
     <axis xyz="0 0 1"/>
   </joint>
@@ -79,5 +94,5 @@
       <origin xyz="0 0 0" rpy="0 0 0"/>
       <geometry>
-        <cylinder length="0.018" radius="0.033"/>
+        <cylinder length="0.018" radius="${wheel_radius}"/>
       </geometry>
     </collision>
@@ -91,5 +106,5 @@
     <parent link="base_link"/>
     <child link="wheel_right_link"/>
-    <origin xyz="0.0 -0.080 0.023" rpy="-1.57 0 0"/>
+    <origin xyz="0.0 -${track_width/2} 0.023" rpy="-1.57 0 0"/>
     <axis xyz="0 0 1"/>
   </joint>
@@ -105,5 +120,5 @@
       <origin xyz="0 0 0" rpy="0 0 0"/>
       <geometry>
-        <cylinder length="0.018" radius="0.033"/>
+        <cylinder length="0.018" radius="${wheel_radius}"/>
       </geometry>
     </collision>

Commit message: Fixed xacro if

File: nuturtle_description/urdf/turtlebot3_burger.urdf.xacro (robot description, xacro)
@@ -63,9 +63,9 @@
       <origin xyz="-0.032 0 0.070" rpy="0 0 0"/>
       <geometry>
-        <xacro:if value="${collision_radius &lt; 0}">
+        <xacro:if value = "${collision_radius &gt; 0.0}">
+          <cylinder length="0.143" radius="${collision_radius}"/>
+        </xacro:if>
+        <xacro:if value = "${collision_radius &lt; 0.0}">
           <box size="0.140 0.140 0.143"/>
-        </xacro:if>
-        <xacro:if value="${collision_radius &gt; 0}">
-          <cylinder length="0.143" radius="${collision_radius}" />
         </xacro:if>
       </geometry>

Commit message: Got color changing with launch

File: nuturtle_description/urdf/turtlebot3_burger.urdf.xacro (robot description, xacro)
@@ -15,4 +15,5 @@
   <xacro:property name="encoder_ticks_per_rad" value="${ros_parameters['encoder_ticks_per_rad']}" />
   <xacro:property name="collision_radius" value="${ros_parameters['collision_radius']}" />
+  <xacro:arg name="color" default="purple" />
   <!-- Init colour -->
   <material name="black">
@@ -21,4 +22,8 @@
   <material name="dark">
     <color rgba="0.3 0.3 0.3 1.0"/>
+  </material>
+  <!-- LSU Purple -->
+  <material name="purple">
+    <color rgba="0.27451 0.113725 0.486275 1.0"/>
   </material>
   <material name="light_black">
@@ -58,5 +63,5 @@
         <mesh filename="package://nuturtle_description/meshes/burger_base.stl" scale="0.001 0.001 0.001"/>
       </geometry>
-      <material name="light_black"/>
+      <material name="$(arg color)"/>
     </visual>
     <collision>

Commit message: Created xml launch file to launch multiple robots at once

File: nuturtle_description/urdf/turtlebot3_burger.urdf.xacro (robot description, xacro)
@@ -52,5 +52,5 @@
   </material>
   <link name="base_footprint"/>
-  <joint name="base_joint" type="fixed">
+  <joint name="zbase_joint" type="fixed">
     <parent link="base_footprint"/>
     <child link="base_link"/>
